Commit message: changed collision box of feet to be short and wide

File: src/adherent/model/iCubGazeboSimpleCollisionsV2_5_xsens/iCubGazeboSimpleCollisionsV2_5_xsens.urdf (robot description, URDF)
Before this commit: robot iCubGazeboSimpleCollisionsV2_5_xsens, 65 links, 64 joints
Links:
- link l_foot: geometry collision box size=0.072 0.1 0.001; visual mesh filename=file://meshes/simmechanics/sim_sea_2-5_l_sole_prt-binary.stl scale=0.001 0.001 0.001
- link r_foot: geometry collision box size=0.072 0.1 0.001; visual mesh filename=file://meshes/simmechanics/sim_sea_2-5_r_sole_prt-binary.stl scale=0.001 0.001 0.001
